Commit message: Un-broke Gazebo

File: install/r6_d9/share/r6_d9/description/gazebo_control.xacro (robot description, xacro)
@@ -1 +1 @@
-/home/easz/r2_ws/src/r6_d9/description/gazebo_control.xacro
+/home/easz/Ros2-R2/src/r6_d9/description/gazebo_control.xacro

File: install/r6_d9/share/r6_d9/description/inertial_macros.xacro (robot description, xacro)
@@ -1 +1 @@
-/home/easz/r2_ws/src/r6_d9/description/inertial_macros.xacro
+/home/easz/Ros2-R2/src/r6_d9/description/inertial_macros.xacro

File: install/r6_d9/share/r6_d9/description/lidar.xacro (robot description, xacro)
@@ -1 +1 @@
-/home/easz/r2_ws/src/r6_d9/description/lidar.xacro
+/home/easz/Ros2-R2/src/r6_d9/description/lidar.xacro

File: install/r6_d9/share/r6_d9/description/robot.urdf.xacro (robot description, xacro)
@@ -1 +1 @@
-/home/easz/r2_ws/src/r6_d9/description/robot.urdf.xacro
+/home/easz/Ros2-R2/src/r6_d9/description/robot.urdf.xacro

File: install/r6_d9/share/r6_d9/description/robot_core.xacro (robot description, xacro)
@@ -1 +1 @@
-/home/easz/r2_ws/src/r6_d9/description/robot_core.xacro
+/home/easz/Ros2-R2/src/r6_d9/description/robot_core.xacro

File: install/r6_d9/share/r6_d9/description/ros2_control.xacro (robot description, xacro)
@@ -1 +1 @@
-/home/easz/r2_ws/src/r6_d9/description/ros2_control.xacro
+/home/easz/Ros2-R2/src/r6_d9/description/ros2_control.xacro

File: src/r6_d9/description/ros2_control.xacro (robot description, xacro)
@@ -1,57 +1,61 @@
 <?xml version="1.0"?>
 <robot xmlns:xacro="http://www.ros.org/wiki/xacro">
-    <ros2_control name="RealRobot" type="system">
-        <hardware>
-            <plugin>diffdrive_arduino/DiffDriveArduinoHardware</plugin>
-            <param name="left_wheel_name">left_wheel_joint</param>
-            <param name="right_wheel_name">right_wheel_joint</param>
-            <param name="loop_rate">30</param>
-            <param name="device">/dev/ttyACM0</param>
-            <param name="baud_rate">57600</param>
-            <param name="timeout_ms">1000</param>
-            <param name="enc_counts_per_rev">2495</param>
-        </hardware>
-        <joint name="left_wheel_joint">
-            <command_interface name="velocity">
-                <param name="min">-10</param>
-                <param name="max">10</param>
-            </command_interface>
-            <state_interface name="position"/>
-            <state_interface name="velocity"/>
-        </joint>
-        <joint name="right_wheel_joint">
-            <command_interface name="velocity">
-                <param name="min">-10</param>
-                <param name="max">10</param>
-            </command_interface>
-            <state_interface name="position"/>
-            <state_interface name="velocity"/>
-        </joint>
-    </ros2_control>
-    <!-- <ros2_control name="GazeboSystem" type="system">
-        <hardware>
-            <plugin>gazebo_ros2_control/GazeboSystem</plugin>
-        </hardware>
-        <joint name="left_wheel_joint">
-            <command_interface name="velocity">
-                <param name="min">-10</param>
-                <param name="max">10</param>
-            </command_interface>
-            <state_interface name="velocity"/>
-            <state_interface name="position"/>
-        </joint>
-        <joint name="right_wheel_joint">
-            <command_interface name="velocity">
-                <param name="min">-10</param>
-                <param name="max">10</param>
-            </command_interface>
-            <state_interface name="velocity"/>
-            <state_interface name="position"/>
-        </joint>
-    </ros2_control> -->
+    <xacro:unless value="$(arg use_sim_mode)">
+        <ros2_control name="RealRobot" type="system">
+            <hardware>
+                <plugin>diffdrive_arduino/DiffDriveArduinoHardware</plugin>
+                <param name="left_wheel_name">left_wheel_joint</param>
+                <param name="right_wheel_name">right_wheel_joint</param>
+                <param name="loop_rate">30</param>
+                <param name="device">/dev/ttyACM0</param>
+                <param name="baud_rate">57600</param>
+                <param name="timeout_ms">1000</param>
+                <param name="enc_counts_per_rev">2495</param>
+            </hardware>
+            <joint name="left_wheel_joint">
+                <command_interface name="velocity">
+                    <param name="min">-10</param>
+                    <param name="max">10</param>
+                </command_interface>
+                <state_interface name="position"/>
+                <state_interface name="velocity"/>
+            </joint>
+            <joint name="right_wheel_joint">
+                <command_interface name="velocity">
+                    <param name="min">-10</param>
+                    <param name="max">10</param>
+                </command_interface>
+                <state_interface name="position"/>
+                <state_interface name="velocity"/>
+            </joint>
+        </ros2_control>
+    </xacro:unless>
+    <xacro:if value="$(arg use_sim_mode)">
+        <ros2_control name="GazeboSystem" type="system">
+            <hardware>
+                <plugin>gazebo_ros2_control/GazeboSystem</plugin>
+            </hardware>
+            <joint name="left_wheel_joint">
+                <command_interface name="velocity">
+                    <param name="min">-10</param>
+                    <param name="max">10</param>
+                </command_interface>
+                <state_interface name="velocity"/>
+                <state_interface name="position"/>
+            </joint>
+            <joint name="right_wheel_joint">
+                <command_interface name="velocity">
+                    <param name="min">-10</param>
+                    <param name="max">10</param>
+                </command_interface>
+                <state_interface name="velocity"/>
+                <state_interface name="position"/>
+            </joint>
+        </ros2_control>
+    </xacro:if>
     <gazebo>
         <plugin name="gazebo_ros2_control" filename="libgazebo_ros2_control.so">
             <parameters>$(find r6_d9)/config/my_controllers.yaml</parameters>
-            <!-- <parameters>$(find articubot_one)/config/gaz_ros2_ctl_use_sim.yaml</parameters> -->
+            <parameters>$(find r6_d9)/config/gaz_ros2_ctl_use_sim.yaml</parameters>
         </plugin>
     </gazebo>
