Commit message: Got slam working?

File: src/r6_d9/description/lidar.xacro (robot description, xacro)
@@ -3,8 +3,8 @@
     <joint name="lidar_joint" type="fixed">
         <parent link="chassis"/>
-        <child link="base_laser"/>
+        <child link="laser_frame"/>
         <origin xyz="-0.045 0.0 0.13" rpy="0.0 -0.35 0.0"/>
     </joint>
-    <link name="base_laser">
+    <link name="laser_frame">
         <visual>
             <geometry>
@@ -22,5 +22,5 @@
         </xacro:inertial_cylinder>
     </link>
-    <gazebo reference="base_laser">
+    <gazebo reference="laser_frame">
         <material>Gazebo/Black</material>
         <sensor name="laser" type="ray">

File: src/r6_d9/description/robot_core.xacro (robot description, xacro)
@@ -10,4 +10,11 @@
     <link name="base_link">
     </link>
+    <joint name="base_footprint_joint" type="fixed">
+        <parent link="base_link"/>
+        <child link="base_footprint"/>
+        <origin xyz="0.0 0.0 0.0" rpy="0.0 0.0 0.0"/>
+    </joint>
+    <link name="base_footprint">
+    </link>
     <!-- Chassis Joint -->
     <joint name="chassis_joint" type="fixed">

File: src/r6_d9/description/ros2_control.xacro (robot description, xacro)
@@ -41,6 +41,6 @@
                     <param name="max">10</param>
                 </command_interface>
+                <state_interface name="position"/>
                 <state_interface name="velocity"/>
-                <state_interface name="position"/>
             </joint>
             <joint name="right_wheel_joint">
@@ -49,6 +49,6 @@
                     <param name="max">10</param>
                 </command_interface>
+                <state_interface name="position"/>
                 <state_interface name="velocity"/>
-                <state_interface name="position"/>
             </joint>
         </ros2_control>

Commit message: minor lidar changes

File: src/r6_d9/description/lidar.xacro (robot description, xacro)
@@ -4,5 +4,5 @@
         <parent link="chassis"/>
         <child link="laser_frame"/>
-        <origin xyz="-0.045 0.0 0.13" rpy="0.0 -0.35 0.0"/>
+        <origin xyz="-0.045 0.0 0.13" rpy="0.0 -0.50 0.0"/>
     </joint>
     <link name="laser_frame">
@@ -19,5 +19,5 @@
         </collision>
         <xacro:inertial_cylinder mass="0.1" length="0.036" radius="0.0165">
-            <origin xyz="-0.045 0.0 0.13" rpy="0 -0.35 0"/>
+            <origin xyz="-0.045 0.0 0.13" rpy="0 -0.50 0"/>
         </xacro:inertial_cylinder>
     </link>

File: src/r6_d9/description/robot_core.xacro (robot description, xacro)
@@ -97,5 +97,5 @@
         <parent link="base_link"/>
         <child link="left_wheel"/>
-        <origin xyz="0.0 -0.145 0.0" rpy="${pi/2} 0.0 0.0"/>
+        <origin xyz="0.0 0.145 0.0" rpy="-${pi/2} 0.0 0.0"/>
         <axis xyz="0.0 0.0 1.0"/>
     </joint>
@@ -125,5 +125,5 @@
         <parent link="base_link"/>
         <child link="right_wheel"/>
-        <origin xyz="0.0 0.145 0.0" rpy="-${pi/2} 0.0 0.0"/>
+        <origin xyz="0.0 -0.145 0.0" rpy="${pi/2} 0.0 0.0"/>
         <axis xyz="0.0 0.0 -1.0"/>
     </joint>

Commit message: nav should be working

File: src/r6_d9/description/lidar.xacro (robot description, xacro)
@@ -3,8 +3,8 @@
     <joint name="lidar_joint" type="fixed">
         <parent link="chassis"/>
-        <child link="laser_frame"/>
+        <child link="base_laser"/>
         <origin xyz="-0.045 0.0 0.13" rpy="0.0 -0.50 0.0"/>
     </joint>
-    <link name="laser_frame">
+    <link name="base_laser">
         <visual>
             <geometry>
@@ -22,5 +22,5 @@
         </xacro:inertial_cylinder>
     </link>
-    <gazebo reference="laser_frame">
+    <gazebo reference="base_laser">
         <material>Gazebo/Black</material>
         <sensor name="laser" type="ray">
@@ -46,5 +46,5 @@
                 </ros>
                 <output_type>sensor_msgs/LaserScan</output_type>
-                <frame_name>laser_frame</frame_name>
+                <frame_name>base_laser</frame_name>
             </plugin>
         </sensor>

Commit message: nah

File: src/r6_d9/description/lidar.xacro (robot description, xacro)
@@ -3,8 +3,8 @@
     <joint name="lidar_joint" type="fixed">
         <parent link="chassis"/>
-        <child link="laser_frame"/>
+        <child link="base_laser"/>
         <origin xyz="-0.045 0.0 0.13" rpy="0.0 -0.50 0.0"/>
     </joint>
-    <link name="laser_frame">
+    <link name="base_laser">
         <visual>
             <geometry>
@@ -22,5 +22,5 @@
         </xacro:inertial_cylinder>
     </link>
-    <gazebo reference="laser_frame">
+    <gazebo reference="base_laser">
         <material>Gazebo/Black</material>
         <sensor name="laser" type="ray">

Commit message: changes on the robot

File: src/r6_d9/description/lidar.xacro (robot description, xacro)
@@ -4,5 +4,5 @@
         <parent link="chassis"/>
         <child link="base_laser"/>
-        <origin xyz="-0.045 0.0 0.13" rpy="0.0 -0.50 0.0"/>
+        <origin xyz="-0.045 0.0 0.13" rpy="${pi} -3.65 0"/>
     </joint>
     <link name="base_laser">

Commit message: minor changes

File: src/r6_d9/description/lidar.xacro (robot description, xacro)
@@ -4,5 +4,5 @@
         <parent link="chassis"/>
         <child link="base_laser"/>
-        <origin xyz="-0.045 0.0 0.13" rpy="0.0 -0.50 0.0"/>
+        <origin xyz="-0.045 0.0 0.13" rpy="0.0 -0.50 ${pi}"/>
     </joint>
     <link name="base_laser">
